File: driver.kicad_sch (KiCad schematic)
At the start: 29 parts, among them J1 FAN_TACH, J2 FAN_PWM, J3 HF1004E, Q1 BSS138, U1 MP2315SGJ-Z

Commit message: add datasheet
Parts:
- removed C1: 25V 10uF, Capacitor_SMD:C_1206_3216Metric_Pad1.33x1.80mm_HandSolder, symbol Device:C
- removed J1: FAN_TACH, Connector_PinHeader_2.54mm:PinHeader_1x01_P2.54mm_Horizontal, symbol Connector:Conn_01x01_Pin
- removed J2: FAN_PWM, Connector_PinHeader_2.54mm:PinHeader_1x01_P2.54mm_Horizontal, symbol Connector:Conn_01x01_Pin
- removed J3: HF1004E, Connector_PinHeader_2.54mm:PinHeader_1x04_P2.54mm_Vertical, symbol Connector:Conn_01x04_Socket
- removed Q1: BSS138, Package_TO_SOT_SMD:SOT-23, symbol Transistor_FET:BSS138
- removed R1: 2.2K, Resistor_SMD:R_0805_2012Metric_Pad1.20x1.40mm_HandSolder, symbol Device:R
- removed R2: 4.7K, Resistor_SMD:R_0805_2012Metric_Pad1.20x1.40mm_HandSolder, symbol Device:R
- removed R3: 27K, Resistor_SMD:R_0805_2012Metric_Pad1.20x1.40mm_HandSolder, symbol Device:R
- removed R4: 10K, Resistor_SMD:R_0805_2012Metric_Pad1.20x1.40mm_HandSolder, symbol Device:R
- removed TH1: KTY85, Diode_SMD:D_MiniMELF, symbol Sensor_Temperature:KTY85
- R1: renamed from R9; value 499K -> 100K
- renumbered C2 to C1, C3 to C2, C4 to C3, C5 to C4, C6 to C5, C8 to C6, C9 to C7, C10 to C8, C7 to C9, R8 to R2, R7 to R3, R11 to R4, R10 to R5, R5 to R6, R6 to R7
