File: mp2236_power_driver/mp2236_power_driver.kicad_pcb (KiCad board)
At the start: 2 copper layers, 29.9 x 20 mm, 17 parts, among them U1 MP2236CGJ-Z

Commit message: version 1.0
Parts:
- added J1: VIN, power_driver:3mmx3mm power pad, F.Cu at (112.0, 78.0)
- added J2: GND, power_driver:3mmx3mm power pad, F.Cu at (116.0, 62.0)
- added J3: VOUT, power_driver:3mmx3mm power pad, F.Cu at (138.0, 78.0)
- added J4: GND, power_driver:3mmx3mm power pad, F.Cu at (112.0, 62.0)
- moved R5 13.0 mm to (115.2, 71.5), turned to 90 degrees
- moved C9 10.1 mm to (125.5, 62.2), turned to -135 degrees
- moved R3 4.28 mm to (122.4, 62.2), turned to -135 degrees
- moved D1 2.77 mm to (111.9, 71.3)
- moved C5 2.24 mm to (128.0, 64.3), turned to -45 degrees
- moved R1 2.10 mm to (118.1, 73.5)
- moved R4 1.13 mm to (116.2, 66.2)
- moved C4 0.83 mm to (118.1, 69.5)
- moved C3 0.51 mm to (121.2, 73.5)
- moved C1 0.34 mm to (121.7, 78.5)
- moved C2 0.34 mm to (121.7, 76.0)
- moved R2 0.28 mm to (125.2, 65.7), turned to 45 degrees
- moved L1 0.10 mm to (133.9, 67.5)
Routing:
- net GND: track 37.8 -> 13.8 mm, vias 56 -> 59
- net /SW: track 18.1 -> 35.9 mm
- net +12V: track 20.4 -> 3.79 mm
- net +5V: track 48.2 -> 31.8 mm
- net /VCC: track 4.94 -> 10.1 mm
- net /BST: track 2.78 -> 0.00 mm
- net Net-(U1-EN): track 17.6 -> 16.8 mm
- net /FB: track 6.64 -> 7.28 mm
- added copper zone on F.Cu, net /BST
- added copper zone on F.Cu, net /FB
Other:
- board size 29.9 x 20 mm -> 30 x 20 mm
- board text added: "+VIN"
- board text added: "+VOUT"
- board text added: "GND"
- board text added: "MP2236 DCDC MODULE VERSION: 1.0 DATE: 2024-12-11"
