File: mp2236_power_driver/mp2236_power_driver.kicad_sch (KiCad schematic)
At the start: 17 parts, among them U1 MP2236CGJ-Z

Commit message: version 1.0
Parts:
- added J1: VIN, power_driver:3mmx3mm power pad, symbol Connector:Conn_01x01_Pin
- added J2, J4: GND, power_driver:3mmx3mm power pad, symbol Connector:Conn_01x01_Pin
- added J3: VOUT, power_driver:3mmx3mm power pad, symbol Connector:Conn_01x01_Pin
Connections:
- net +12V: now also J1.1 (Pin_1)
- net +5V: now also J3.1 (Pin_1)
- net GND: now also J2.1 (Pin_1), J4.1 (Pin_1)
