File: mp2236_dcdc_module/mp2236_power_driver.kicad_sch (KiCad schematic)
At the start: 21 parts, among them J1 VIN, J2 GND, J3 VOUT, J4 GND, U1 MP2236CGJ-Z

Commit message: mp2236 power module v1.1
Parts:
- removed J1: VIN, power_driver:3mmx3mm power pad, symbol Connector:Conn_01x01_Pin
- removed J2, J4: GND, power_driver:3mmx3mm power pad, symbol Connector:Conn_01x01_Pin
- removed J3: VOUT, power_driver:3mmx3mm power pad, symbol Connector:Conn_01x01_Pin
- added J1, J2: Conn_01x02_Socket, power_driver:4mmx5mm_2x18.0mm power pad, symbol Connector:Conn_01x02_Socket
- added LED1: LED_0603_Green, PCM_LED_SMD_AKL:LED_0603_1608Metric, symbol PCM_LED_AKL:LED_0603_Green
- added R6: 5.1K, Resistor_SMD:R_0603_1608Metric, symbol Device:R
- C1, C2: footprint Capacitor_SMD:C_1206_3216Metric_Pad1.33x1.80mm_HandSolder -> Capacitor_SMD:C_1206_3216Metric
- C3, C4, C5, C9: footprint Capacitor_SMD:C_0805_2012Metric_Pad1.18x1.45mm_HandSolder -> Capacitor_SMD:C_0603_1608Metric
- C6, C7, C8: footprint Capacitor_SMD:C_1206_3216Metric_Pad1.33x1.80mm_HandSolder -> Capacitor_SMD:C_0805_2012Metric
- R1, R2, R3, R4, R5: footprint Resistor_SMD:R_0805_2012Metric_Pad1.20x1.40mm_HandSolder -> Resistor_SMD:R_0603_1608Metric
- U1: footprint Package_TO_SOT_SMD:TSOT-23-8_HandSoldering -> PCM_Package_TO_SOT_SMD_AKL:TSOT-23-8
Connections:
- net +12V: now also J1.1 (Pin_1)
- net +5V: now also J2.1 (Pin_1), R6.1
- net GND: now also J1.2 (Pin_2), J2.2 (Pin_2), LED1.1 (K)
- new net: LED1.2 (A), R6.2
Other:
- title: MP2236电源模块 -> MP2236电源模块 12V转5V
